File: BlueRov_pcb/BlueRov_pcb.kicad_pcb (KiCad board)
At the start: 2 copper layers, 73.7 x 59.7 mm, 19 parts, among them J1 Vin, J10 Conn_02x19_Odd_Even, J11 Conn_01x04, J3 Conn_01x03, J4 Conn_01x03, J5 Conn_01x03, J6 Conn_01x03, J7 Conn_02x19_Odd_Even, J8 Conn_01x03, J9 Conn_01x04, U1 L7805

Commit message: szyk pcb
Parts:
- removed the C1 at (204.1, 119.4)
- removed the C2 at (198.1, 122.6)
- removed the C3 at (209.5, 122.6)
- removed the C4 at (208.0, 128.3)
- removed the D1 at (184.2, 131.1)
- removed the J1 at (190.5, 127.0)
- removed the J10 at (236.2, 86.4)
- removed the J11 at (227.3, 94.0)
- removed the J3 at (184.2, 86.4)
- removed the J4 at (194.3, 86.4)
- removed the J5 at (224.8, 86.4)
- removed the J6 at (214.6, 86.4)
- removed the J7 at (175.3, 86.4)
- removed the J8 at (204.5, 86.4)
- removed the J9 at (185.4, 94.0)
- removed the R1 at (183.9, 124.5)
- removed the R2 at (183.9, 127.4)
- removed the R3 at (181.6, 131.1)
- removed the U1 at (201.9, 113.7)
- added C1: 100n, Capacitor_SMD:C_0805_2012Metric_Pad1.15x1.40mm_HandSolder, F.Cu at (215.9, 170.5)
- added C1: 100n, Capacitor_SMD:C_0805_2012Metric_Pad1.15x1.40mm_HandSolder, F.Cu at (68.6, 165.9)
- added C1: 100n, Capacitor_SMD:C_0805_2012Metric_Pad1.15x1.40mm_HandSolder, F.Cu at (215.2, 73.2)
- added C1: 100n, Capacitor_SMD:C_0805_2012Metric_Pad1.15x1.40mm_HandSolder, F.Cu at (68.2, 68.7)
- added C2: 22u, Capacitor_THT:CP_Radial_D5.0mm_P2.50mm, F.Cu at (210.0, 173.7)
- added C2: 22u, Capacitor_THT:CP_Radial_D5.0mm_P2.50mm, F.Cu at (62.6, 169.1)
- added C2: 22u, Capacitor_THT:CP_Radial_D5.0mm_P2.50mm, F.Cu at (209.2, 76.3)
- added C2: 22u, Capacitor_THT:CP_Radial_D5.0mm_P2.50mm, F.Cu at (62.2, 71.9)
- added C3: 22u, Capacitor_THT:CP_Radial_D5.0mm_P2.50mm, F.Cu at (221.4, 173.7)
- added C3: 22u, Capacitor_THT:CP_Radial_D5.0mm_P2.50mm, F.Cu at (74.0, 169.1)
- added C3: 22u, Capacitor_THT:CP_Radial_D5.0mm_P2.50mm, F.Cu at (220.6, 76.3)
- added C3: 22u, Capacitor_THT:CP_Radial_D5.0mm_P2.50mm, F.Cu at (73.6, 71.9)
- added C4: 100n, Capacitor_SMD:C_0805_2012Metric_Pad1.15x1.40mm_HandSolder, F.Cu at (219.9, 179.4)
- added C4: 100n, Capacitor_SMD:C_0805_2012Metric_Pad1.15x1.40mm_HandSolder, F.Cu at (72.5, 174.8)
- added C4: 100n, Capacitor_SMD:C_0805_2012Metric_Pad1.15x1.40mm_HandSolder, F.Cu at (219.1, 82.0)
- added C4: 100n, Capacitor_SMD:C_0805_2012Metric_Pad1.15x1.40mm_HandSolder, F.Cu at (72.1, 77.6)
- added D1: LED, Capacitor_SMD:C_0805_2012Metric_Pad1.15x1.40mm_HandSolder, F.Cu at (196.0, 182.2)
- added D1: LED, Capacitor_SMD:C_0805_2012Metric_Pad1.15x1.40mm_HandSolder, F.Cu at (48.6, 177.6)
- added D1: LED, Capacitor_SMD:C_0805_2012Metric_Pad1.15x1.40mm_HandSolder, F.Cu at (195.2, 84.8)
- added D1: LED, Capacitor_SMD:C_0805_2012Metric_Pad1.15x1.40mm_HandSolder, F.Cu at (48.3, 80.4)
- added J1: Vin, Connector_Molex:Molex_Mini-Fit_Jr_5566-02A_2x01_P4.20mm_Vertical, F.Cu at (202.4, 178.1)
- added J1: Vin, Connector_Molex:Molex_Mini-Fit_Jr_5566-02A_2x01_P4.20mm_Vertical, F.Cu at (55.0, 173.5)
- added J1: Vin, Connector_Molex:Molex_Mini-Fit_Jr_5566-02A_2x01_P4.20mm_Vertical, F.Cu at (201.6, 80.8)
- added J1: Vin, Connector_Molex:Molex_Mini-Fit_Jr_5566-02A_2x01_P4.20mm_Vertical, F.Cu at (54.6, 76.3)
- added J10: Conn_02x19_Odd_Even, Connector_PinSocket_2.54mm:PinSocket_2x19_P2.54mm_Vertical, B.Cu at (248.1, 137.5)
- added J10: Conn_02x19_Odd_Even, Connector_PinSocket_2.54mm:PinSocket_2x19_P2.54mm_Vertical, B.Cu at (100.7, 132.9)
- added J10: Conn_02x19_Odd_Even, Connector_PinSocket_2.54mm:PinSocket_2x19_P2.54mm_Vertical, B.Cu at (247.3, 40.1)
- added J10: Conn_02x19_Odd_Even, Connector_PinSocket_2.54mm:PinSocket_2x19_P2.54mm_Vertical, B.Cu at (100.3, 35.7)
- added J11: Conn_01x04, Connector_PinHeader_2.54mm:PinHeader_1x04_P2.54mm_Vertical, F.Cu at (239.2, 145.1)
- added J11: Conn_01x04, Connector_PinHeader_2.54mm:PinHeader_1x04_P2.54mm_Vertical, F.Cu at (91.8, 140.5)
- added J11: Conn_01x04, Connector_PinHeader_2.54mm:PinHeader_1x04_P2.54mm_Vertical, F.Cu at (238.4, 47.8)
- added J11: Conn_01x04, Connector_PinHeader_2.54mm:PinHeader_1x04_P2.54mm_Vertical, F.Cu at (91.4, 43.3)
- added J3: Conn_01x03, Connector_PinHeader_2.54mm:PinHeader_1x03_P2.54mm_Horizontal, F.Cu at (196.0, 137.5)
- added J3: Conn_01x03, Connector_PinHeader_2.54mm:PinHeader_1x03_P2.54mm_Horizontal, F.Cu at (48.6, 132.9)
- added J3: Conn_01x03, Connector_PinHeader_2.54mm:PinHeader_1x03_P2.54mm_Horizontal, F.Cu at (195.2, 40.1)
- added J3: Conn_01x03, Connector_PinHeader_2.54mm:PinHeader_1x03_P2.54mm_Horizontal, F.Cu at (48.3, 35.7)
- added J4: Conn_01x03, Connector_PinHeader_2.54mm:PinHeader_1x03_P2.54mm_Horizontal, F.Cu at (206.2, 137.5)
- added J4: Conn_01x03, Connector_PinHeader_2.54mm:PinHeader_1x03_P2.54mm_Horizontal, F.Cu at (58.8, 132.9)
- added J4: Conn_01x03, Connector_PinHeader_2.54mm:PinHeader_1x03_P2.54mm_Horizontal, F.Cu at (205.4, 40.1)
- added J4: Conn_01x03, Connector_PinHeader_2.54mm:PinHeader_1x03_P2.54mm_Horizontal, F.Cu at (58.4, 35.7)
- added J5: Conn_01x03, Connector_PinHeader_2.54mm:PinHeader_1x03_P2.54mm_Horizontal, F.Cu at (236.7, 137.5)
- added J5: Conn_01x03, Connector_PinHeader_2.54mm:PinHeader_1x03_P2.54mm_Horizontal, F.Cu at (89.3, 132.9)
- added J5: Conn_01x03, Connector_PinHeader_2.54mm:PinHeader_1x03_P2.54mm_Horizontal, F.Cu at (235.9, 40.1)
- added J5: Conn_01x03, Connector_PinHeader_2.54mm:PinHeader_1x03_P2.54mm_Horizontal, F.Cu at (88.9, 35.7)
- added J6: Conn_01x03, Connector_PinHeader_2.54mm:PinHeader_1x03_P2.54mm_Horizontal, F.Cu at (226.5, 137.5)
- added J6: Conn_01x03, Connector_PinHeader_2.54mm:PinHeader_1x03_P2.54mm_Horizontal, F.Cu at (79.1, 132.9)
- added J6: Conn_01x03, Connector_PinHeader_2.54mm:PinHeader_1x03_P2.54mm_Horizontal, F.Cu at (225.7, 40.1)
- added J6: Conn_01x03, Connector_PinHeader_2.54mm:PinHeader_1x03_P2.54mm_Horizontal, F.Cu at (78.7, 35.7)
- added J7: Conn_02x19_Odd_Even, Connector_PinSocket_2.54mm:PinSocket_2x19_P2.54mm_Vertical, B.Cu at (187.1, 137.5)
- added J7: Conn_02x19_Odd_Even, Connector_PinSocket_2.54mm:PinSocket_2x19_P2.54mm_Vertical, B.Cu at (39.8, 132.9)
- added J7: Conn_02x19_Odd_Even, Connector_PinSocket_2.54mm:PinSocket_2x19_P2.54mm_Vertical, B.Cu at (186.4, 40.1)
- added J7: Conn_02x19_Odd_Even, Connector_PinSocket_2.54mm:PinSocket_2x19_P2.54mm_Vertical, B.Cu at (39.4, 35.7)
- added J8: Conn_01x03, Connector_PinHeader_2.54mm:PinHeader_1x03_P2.54mm_Horizontal, F.Cu at (216.3, 137.5)
- added J8: Conn_01x03, Connector_PinHeader_2.54mm:PinHeader_1x03_P2.54mm_Horizontal, F.Cu at (69.0, 132.9)
- added J8: Conn_01x03, Connector_PinHeader_2.54mm:PinHeader_1x03_P2.54mm_Horizontal, F.Cu at (215.6, 40.1)
- added J8: Conn_01x03, Connector_PinHeader_2.54mm:PinHeader_1x03_P2.54mm_Horizontal, F.Cu at (68.6, 35.7)
- added J9: Conn_01x04, Connector_PinHeader_2.54mm:PinHeader_1x04_P2.54mm_Vertical, F.Cu at (197.3, 145.1)
- added J9: Conn_01x04, Connector_PinHeader_2.54mm:PinHeader_1x04_P2.54mm_Vertical, F.Cu at (49.9, 140.5)
- added J9: Conn_01x04, Connector_PinHeader_2.54mm:PinHeader_1x04_P2.54mm_Vertical, F.Cu at (196.5, 47.8)
- added J9: Conn_01x04, Connector_PinHeader_2.54mm:PinHeader_1x04_P2.54mm_Vertical, F.Cu at (49.5, 43.3)
- added R1: 15k, Resistor_SMD:R_0805_2012Metric_Pad1.15x1.40mm_HandSolder, F.Cu at (195.8, 175.6)
- added R1: 15k, Resistor_SMD:R_0805_2012Metric_Pad1.15x1.40mm_HandSolder, F.Cu at (48.4, 171.0)
- added R1: 15k, Resistor_SMD:R_0805_2012Metric_Pad1.15x1.40mm_HandSolder, F.Cu at (195.0, 78.2)
- added R1: 15k, Resistor_SMD:R_0805_2012Metric_Pad1.15x1.40mm_HandSolder, F.Cu at (48.0, 73.8)
- added R2: 3k, Resistor_SMD:R_0805_2012Metric_Pad1.15x1.40mm_HandSolder, F.Cu at (195.8, 178.5)
- added R2: 3k, Resistor_SMD:R_0805_2012Metric_Pad1.15x1.40mm_HandSolder, F.Cu at (48.4, 173.9)
- added R2: 3k, Resistor_SMD:R_0805_2012Metric_Pad1.15x1.40mm_HandSolder, F.Cu at (195.0, 81.2)
- added R2: 3k, Resistor_SMD:R_0805_2012Metric_Pad1.15x1.40mm_HandSolder, F.Cu at (48.0, 76.7)
- added R3: 470, Resistor_SMD:R_0805_2012Metric_Pad1.15x1.40mm_HandSolder, F.Cu at (193.5, 182.2)
- added R3: 470, Resistor_SMD:R_0805_2012Metric_Pad1.15x1.40mm_HandSolder, F.Cu at (46.1, 177.6)
- added R3: 470, Resistor_SMD:R_0805_2012Metric_Pad1.15x1.40mm_HandSolder, F.Cu at (192.7, 84.8)
- added R3: 470, Resistor_SMD:R_0805_2012Metric_Pad1.15x1.40mm_HandSolder, F.Cu at (45.7, 80.4)
- added U1: L7805, Package_TO_SOT_SMD:SOT-223-3_TabPin2, F.Cu at (213.8, 164.8)
- added U1: L7805, Package_TO_SOT_SMD:SOT-223-3_TabPin2, F.Cu at (66.4, 160.2)
- added U1: L7805, Package_TO_SOT_SMD:SOT-223-3_TabPin2, F.Cu at (213.0, 67.4)
- added U1: L7805, Package_TO_SOT_SMD:SOT-223-3_TabPin2, F.Cu at (66.0, 63.0)
Routing:
- net +5V: track 72.1 -> 288.4 mm, vias 2 -> 8
- net TIM3_CH3: track 51.6 -> 206.5 mm
- net TIM2_CH2: track 44.3 -> 177.0 mm
- net TIM2_CH1: track 43.2 -> 172.7 mm
- net RO: track 37.7 -> 150.9 mm, vias 1 -> 4
- net DI: track 34.4 -> 137.7 mm, vias 1 -> 4
- net TIM3_CH2: track 34.4 -> 137.7 mm
- net +3V3: track 30.2 -> 120.6 mm, vias 1 -> 4
- net VCC: track 28.8 -> 115.1 mm
- net TIM3_CH1: track 24.0 -> 96.1 mm
- net DE: track 21.1 -> 84.4 mm, vias 1 -> 4
- net GND: track 16.6 -> 66.3 mm, vias 1 -> 4
- net ADC: track 8.31 -> 33.3 mm
- net USER_LED: track 3.81 -> 15.2 mm
- net Net-(D1-Pad2): track 2.54 -> 10.2 mm
Other:
- board size 73.7 x 59.7 mm -> 221.4 x 161.5 mm
